File: sch/periph.sch (KiCad schematic (older format))
At the start: 93 parts, among them P7 PIN, P8 PIN, Q3 QUARTZ, X3 CONN-5S, X5.A1 CONN-7S, X5.B1 CONN-7S, X6 CONN-7S, X7 CONN-7S, X8 CONN-12, X9 CONN-12

Commit message: More precise version. PCB needs a lot of work.
Parts:
- C10, C22: value 100мк -> CAPP
- C11: value 12 -> CAP; footprint MyLib:C_Disc_D7.5_P2.5 -> MyLib_metric:C_Disc_D7.5_P2.5
- C12: value 24 -> CAP; footprint MyLib:C_Disc_D7.5_P2.5 -> MyLib_metric:C_Disc_D7.5_P2.5
- C13: value 47н -> CAP; footprint MyLib:C_Disc_D7.5_P2.5 -> MyLib_metric:C_Disc_D7.5_P2.5
- C23: value 0,47мк -> CAP; footprint MyLib:C_Disc_D7.5_P2.5 -> MyLib_metric:C_Disc_D7.5_P2.5
- C25, C26: value 47мк -> CAPP
- C6: value 1мк -> CAPP
- C9: value 1,5мк -> CAP; footprint MyLib:C_Disc_D7.5_P2.5 -> MyLib_metric:C_Disc_D7.5_P2.5
- D17, D18: footprint MyLib:DIP-40 -> MyLib_metric:DIP-40
- D19, D33, D82, D83: footprint MyLib:DIP-24 -> MyLib_metric:DIP-24
- D34: footprint MyLib:DIP-28 -> MyLib_metric:DIP-28
- D41, D42, D75, D78: footprint MyLib:DIP-14 -> MyLib_metric:DIP-14
- D79, D80, D81: footprint MyLib:DIP-16 -> MyLib_metric:DIP-16
- D84: footprint MyLib:DIP-20 -> MyLib_metric:DIP-20
- D86: footprint MyLib:DIP-8 -> MyLib_metric:DIP-8
- DR2: value 51мкГ -> INDUCTOR
- Q3: footprint MyLib:Crystal_Round_Vertical_5mm -> MyLib_metric:Crystal_Round_Vertical_5mm
- R100, R105: value 1,2к -> 1.2K; footprint MyLib:Resistor_Horizontal_RM7.5mm -> MyLib_metric:Resistor_Horizontal_RM7.5mm
- R114, R115, R116, R117, R118, R119, R120, R121, R122, R129, R130, R33, R34, R36: footprint MyLib:Resistor_Horizontal_RM7.5mm -> MyLib_metric:Resistor_Horizontal_RM7.5mm
- R123: value 2,7к -> RES; footprint MyLib:Resistor_Horizontal_RM7.5mm -> MyLib_metric:Resistor_Horizontal_RM7.5mm
- R126, R132, R82, R83, R84, R85, R86, R87: value 2,7к -> 2K; footprint MyLib:Resistor_Horizontal_RM7.5mm -> MyLib_metric:Resistor_Horizontal_RM7.5mm
- R127, R131: value 6,8к -> 2K; footprint MyLib:Resistor_Horizontal_RM7.5mm -> MyLib_metric:Resistor_Horizontal_RM7.5mm
- R128, R133: value 3,3к -> 2K; footprint MyLib:Resistor_Horizontal_RM7.5mm -> MyLib_metric:Resistor_Horizontal_RM7.5mm
- R17, R21, R22, R23, R88, R89, R90, R91, R92, R93, R94, R95: value 10к -> RES; footprint MyLib:Resistor_Vertical_RM2.5mm -> MyLib_metric:Resistor_Vertical_RM2.5mm
- R35: value 390к -> RES; footprint MyLib:Resistor_Horizontal_RM7.5mm -> MyLib_metric:Resistor_Horizontal_RM7.5mm
- R37: value 10М -> RES; footprint MyLib:Resistor_Horizontal_RM7.5mm -> MyLib_metric:Resistor_Horizontal_RM7.5mm
- R38: value 470к -> RES; footprint MyLib:Resistor_Horizontal_RM7.5mm -> MyLib_metric:Resistor_Horizontal_RM7.5mm
- VD10, VD11, VD13, VD14, VD4, VD6, VD7, VD9: footprint MyLib:Diode_DO-35_SOD27_Horizontal_RM7.5 -> MyLib_metric:Diode_DO-35_SOD27_Horizontal_RM7.5
- X8, X9: footprint MyLib:FB-12 -> MyLib_metric:FB-12

Commit message: IR22 and IR23 symbols updated, part values updated
Parts:
- C10, C22: value CAPP -> 100мк
- C11: value CAP -> 12
- C12: value CAP -> 24
- C13: value CAP -> 47н
- C23: value CAP -> 0,47мк
- C25, C26: value CAPP -> 47мк
- C6: value CAPP -> 1мк
- C9: value CAP -> 1,5мк
- DR2: value INDUCTOR -> 51мкГ
- R100, R105, R36: value 1.2K -> 1,2к
- R123: value RES -> 2,7к
- R126, R132, R82, R83, R84, R85, R86, R87: value 2K -> 2,7к
- R127, R131: value 2K -> 6,8к
- R128, R133: value 2K -> 3,3к
- R17, R21, R22, R23, R88, R89, R90, R91, R92, R93, R94, R95: value RES -> 10к
- R33: value 10K -> 10к
- R35: value RES -> 390к
- R37: value RES -> 10М
- R38: value RES -> 470к
Connections:
- net Z0: now also D84.2 (Q0); no longer D84.5 (Q1)
- net Z1: now also D84.5 (Q1); no longer D84.6 (Q2)
- net Z2: now also D84.6 (Q2); no longer D84.9 (Q3)
- net Z3: now also D84.9 (Q3); no longer D84.12 (Q4)
- net Z4: now also D84.12 (Q4); no longer D84.15 (Q5)
- net Z5: now also D84.15 (Q5); no longer D84.16 (Q6)
- net Z6: now also D84.16 (Q6); no longer D84.19 (Q7)
- net Z7: now also D84.19 (Q7)
Other:
- moved on the sheet: C22, C23, C25, C26, D78A, D78B, D84, DR2, R129, R130, VD10, VD11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
