File: sch/periph.sch (KiCad schematic (older format))
At the start: 93 parts, among them P7 PIN, P8 PIN, Q3 QUARTZ, X3 CONN-5S, X5.A1 CONN-7S, X5.B1 CONN-7S, X6 CONN-7S, X7 CONN-7S, X8 CONN-12, X9 CONN-12

Commit message: Start to move to a bit more affordable components
Parts:
- removed unit 1 of D42
- removed unit 2 of D42
- removed D75: 555ЛА3, MyLib:DIP-14, symbol 555ЛА3
- removed unit 1 of D78
- removed unit 2 of D78
- removed D79: 555ТМ9, MyLib:DIP-16, symbol 555ТМ9
- removed D80: 555ИД10, MyLib:DIP-16, symbol 555ИД10
- removed D81: 555КП7, MyLib:DIP-16, symbol 555КП7
- removed D82, D83: 1802ИР1, MyLib:DIP-24, symbol 1802ИР1
- removed D84: 555ИР23, MyLib:DIP-20, symbol 555ИР23
- removed P7, P8: PIN, MyLib:PIN, symbol PIN
- removed R100, R105: 1,2к, MyLib:Resistor_Horizontal_RM7.5mm, symbol RES
- removed R17, R21, R22, R23, R88, R89, R90, R91, R92, R93, R94, R95: 10к, MyLib:Resistor_Vertical_RM2.5mm, symbol RES
- removed R82, R83, R84, R85, R86, R87: 2,7к, MyLib:Resistor_Horizontal_RM7.5mm, symbol RES
- removed VD9: DIODE_MY, MyLib:Diode_DO-35_SOD27_Horizontal_RM7.5, symbol DIODE_MY
- removed X7: CONN-7S, MyLib:DNR-8F1R, symbol CONN-7S
- removed X8, X9: CONN-12, MyLib:FB-12, symbol CONN-12
- added DD? (x4): 555ЛА3, symbol 555ЛА3
- added G?: BAT, Connect:CR2032H, symbol BAT
- added R17: RES_PACK4_C, MyLib:Resistor_Array_SIP4, symbol RES_PACK4_C
- added R? (x3): 1K, symbol RES
- added R? (x5): 10K, symbol RES
- added R? (x2): 22K, symbol RES
- added R?: RES, MyLib:Resistor_Horizontal_RM7.5mm, symbol RES
- added R?: 2.2K, MyLib:Resistor_Horizontal_RM7.5mm, symbol RES
- added SB?: BUT_OFF, Pin_Headers:Pin_Header_Straight_1x02, symbol BUT_OFF
- added X? (x2): CONN-6S, r_mini_din:Mini_din6, symbol CONN-6S
- added X?: CONN-9, Connect:DB9MC, symbol CONN-9
- C10, C22: value 100мк -> CAPP
- C11: value 12 -> CAP
- C12: value 24 -> CAP
- C13: value 47н -> CAP
- C23: value 0,47мк -> CAP
- C25, C26: value 47мк -> CAPP
- C6: value 1мк -> CAPP
- C9: value 1,5мк -> CAP
- DR2: value 51мкГ -> INDUCTOR
- R114, R115, R116, R117, R118, R119, R120, R121, R122: value 27 -> RES
- R123, R126, R132: value 2,7к -> RES
- R127, R131: value 6,8к -> RES
- R128, R133: value 3,3к -> RES
- R129: value 510 -> RES
- R130: value 220 -> RES
- R33: value 10K -> RES
- R34: value 10k -> RES
- R35: value 390к -> RES
- R36: value 1.2K -> RES
- R37: value 10М -> RES
- R38: value 470к -> RES
Connections:
- net labels added: AGND, KCLK, KDAT, LEFT, MCLK, MDAT, RIGHT, SA, SB, SC, ~BUSRESET, ~EXP
- net labels removed: 1CY, 2CY, KK0, KK1, KK2, KK3, KM0, KM1, KM10, KM11, KM12, KM13, KM14, KM15, KM16, KM17, KM18, KM2, KM3, KM4, KM5, KM6, KM7, KM8, KM9, KRS, KW0, KW1, KW2, KW3, MK0, MK1, MK2, MK3, SABC, SINT, SINT*, Z0, Z1, Z2, Z3, Z4, Z5, Z6, Z7, ~3CY
- wire segments 466 -> 340
- no-connect marks 16 -> 19
Other:
- note added: "+5V"
- note added: "Clock"
- note added: "DCD"
- note added: "DSR"
- note added: "DTR"
- note added: "Data"
- note added: "Keyboard"
- note added: "Mouse"
- note added: "Onboard reset"
- note added: "RI"
- note added: "Shield"
- note removed: "+12V"
- note removed: "KEYBOARD"
- note removed: "KI0"
- note removed: "KI1"
- note removed: "KI2"
- note removed: "KI3"
- note removed: "KI4"
- note removed: "KI5"
- note removed: "KI6"
- note removed: "KI7"
- note removed: "KO0"
- note removed: "KO1"
- note removed: "KO10"
- note removed: "KO2"
- note removed: "KO3"
- note removed: "KO4"
- note removed: "KO5"
- note removed: "KO6"
- note removed: "KO7"
- note removed: "KO8"
- note removed: "KO9"
- note removed: "SBRESET"
- note removed: "VBAT"
- moved on the sheet: C10, C11, C12, C13, C22, C23, C25, C26, C6, C9, D19, D33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
