File: sch/fdc.sch (KiCad schematic (older format))
At the start: 22 parts, among them X4 SLOT-34

Commit message: Start to move to a bit more affordable components
Parts:
- removed R67, R68, R69, R70: 2,7к, MyLib:Resistor_Vertical_RM2.5mm, symbol RES
- removed R71, R72, R73, R74, R75: 1,2к, MyLib:Resistor_Vertical_RM2.5mm, symbol RES
- added R67: RES_PACK4_C, MyLib:Resistor_Array_SIP4, symbol RES_PACK4_C
- added R71: RES_PACK8_C, MyLib:Resistor_Array_SIP5, symbol RES_PACK8_C
- added SA?: SW_OFF, Pin_Headers:Pin_Header_Straight_1x02, symbol SW_OFF
- R76: value 2,7к -> RES
Connections:
- net FP0: now also R71.2
- net FP1: now also R71.3
- net FP2: now also R71.4
- net FP3: now also R71.5
- net GND: now also SA?.1
- net VCC: now also R67.1, R67.1, R67.1, R67.1, R71.1, R71.1, R71.1, R71.1, R71.1
- net WRC: now also R71.6
- net ~INDEX: now also R67.4
- net ~RDATA: now also R67.3
- net ~SIDE: now also SA?.2
- net ~TRAC0: now also R67.2
- net ~WRTPRT: now also R67.5
Other:
- note added: "Force second side"
- moved on the sheet: R76

Commit message: GAL based PLL for FDC
Parts:
- removed D68: 555ТМ9, MyLib:DIP-16, symbol 555ТМ9
- removed D69: 155РЕ3, MyLib:DIP-16, symbol 155РЕ3
- removed R71: RES_PACK8_C, MyLib:Resistor_Array_SIP5, symbol RES_PACK8_C
- added DD?: GAL16V8, symbol GAL16V8
Connections:
- net GND: now also DD?.10 (GND), DD?.11 (OE)
- net RDD: now also DD?.17 (IO5)
- net VCC: now also DD?.20 (VCC)
- net WRC: now also DD?.16 (IO4)
- net at D71.1 (R): now also DD?.18 (IO6)
- net at C18.2, D71.6: now also DD?.2 (I1)
- net at D72.9 (Q1): now also DD?.1 (CLK)
- net at D72.14 (C1): now also DD?.15 (IO3); no longer D73.2 (out)
- no-connect marks 20 -> 31
Other:
- moved on the sheet: C18, D71A, D73A, R67B
