File: sch/gatearray.sch (KiCad schematic (older format))
At the start: 71 parts, among them X2 CONN-7S

Commit message: More precise version. PCB needs a lot of work.
Parts:
- C14: value 100мк -> CAPP
- C15, C16, C17, C4, C5: footprint MyLib:C_Disc_D7.5_P2.5 -> MyLib_metric:C_Disc_D7.5_P2.5
- D26, D28, D32, D49, D50, D51, D52, D53, D54, D55, D56, D59, D87, D88: footprint MyLib:DIP-16 -> MyLib_metric:DIP-16
- D29, D35, D43, D44, D57, D77, D85: footprint MyLib:DIP-14 -> MyLib_metric:DIP-14
- D58, D89: footprint MyLib:DIP-20 -> MyLib_metric:DIP-20
- D60, D61, D62: footprint MyLib:DIP-24 -> MyLib_metric:DIP-24
- DR1: value 91мкГ -> INDUCTOR
- R101, R136, R16, R57, R62, R63, R64, R65, R66, R81: footprint MyLib:Resistor_Horizontal_RM7.5mm -> MyLib_metric:Resistor_Horizontal_RM7.5mm
- R134, R53, R55: value 360 -> RES; footprint MyLib:Resistor_Horizontal_RM7.5mm -> MyLib_metric:Resistor_Horizontal_RM7.5mm
- R28, R29, R30, R31, R32, R47, R48, R49, R50: value 1,2к -> RES; footprint MyLib:Resistor_Vertical_RM2.5mm -> MyLib_metric:Resistor_Vertical_RM2.5mm
- R51: value 1,2к -> 1.2k; footprint MyLib:Resistor_Horizontal_RM7.5mm -> MyLib_metric:Resistor_Horizontal_RM7.5mm
- R52, R54: value 200 -> RES; footprint MyLib:Resistor_Horizontal_RM7.5mm -> MyLib_metric:Resistor_Horizontal_RM7.5mm
- R56: value 200 -> 120; footprint MyLib:Resistor_Horizontal_RM7.5mm -> MyLib_metric:Resistor_Horizontal_RM7.5mm
- R58: value 510 -> RES; footprint MyLib:Resistor_Horizontal_RM7.5mm -> MyLib_metric:Resistor_Horizontal_RM7.5mm
- R59: value 6,8к -> 1.2K; footprint MyLib:Resistor_Horizontal_RM7.5mm -> MyLib_metric:Resistor_Horizontal_RM7.5mm
- R6: value 2,7к -> 15K; footprint MyLib:Resistor_Horizontal_RM7.5mm -> MyLib_metric:Resistor_Horizontal_RM7.5mm
- R60: value 1,2к -> 1.2K; footprint MyLib:Resistor_Horizontal_RM7.5mm -> MyLib_metric:Resistor_Horizontal_RM7.5mm
- R61: value 3,3к -> 1.2K; footprint MyLib:Resistor_Horizontal_RM7.5mm -> MyLib_metric:Resistor_Horizontal_RM7.5mm
- VD12, VD2, VD8: footprint MyLib:Diode_DO-35_SOD27_Horizontal_RM7.5 -> MyLib_metric:Diode_DO-35_SOD27_Horizontal_RM7.5

Commit message: IR22 and IR23 symbols updated, part values updated
Parts:
- C14: value CAPP -> 100мк
- DR1: value INDUCTOR -> 91мкГ
- R134, R53, R55: value RES -> 360
- R28, R29, R30, R31, R32, R47, R48, R49, R50: value RES -> 1,2к
- R51: value 1.2k -> 1,2к
- R52, R54: value RES -> 200
- R56: value 120 -> 200
- R58: value RES -> 510
- R59: value 1.2K -> 6,8к
- R6: value 15K -> 2,7к
- R60: value 1.2K -> 1,2к
- R61: value 1.2K -> 3,3к
Connections:
- net C0: now also D58.2 (Q0); no longer D58.5 (Q1)
- net C1: now also D58.5 (Q1); no longer D58.6 (Q2)
- net C2: now also D58.6 (Q2); no longer D58.9 (Q3)
- net C3: now also D58.9 (Q3); no longer D58.12 (Q4)
- net C4: now also D58.12 (Q4); no longer D58.15 (Q5)
- net C5: now also D58.15 (Q5); no longer D58.16 (Q6)
Other:
- moved on the sheet: D56

Commit message: Board fully redrawn
Changed lines of the file:
@@
 U 1 1 56791C88
 P 3900 1500
+AR Path="/56791C88" Ref="D54"  Part="1"
+AR Path="/5676251A/56791C88" Ref="D54"  Part="1"
 F 0 "D54" H 4450 1650 60  0000 C CNN
 F 1 "555ИД4" H 4450 550 50  0000 C CNN
@@
 Text HLabel 8500 5300 0    60   Input ~ 0
 4M
-Text Label 10400 6100 2    60   ~ 0
-MVI
 Text Label 10400 5700 2    60   ~ 0
 8ST
@@
 Text Label 5800 2500 0    60   ~ 0
 RRC
-Text Label 5800 2600 0    60   ~ 0
-MVI
 Text Label 5800 4300 0    60   ~ 0
 RRC
-Text Label 5800 4400 0    60   ~ 0
-MVI
 $Comp
 L VCC #PWR036
@@
 	5700 2400 5800 2500
 Entry Wire Line
-	5700 2500 5800 2600
-Entry Wire Line
 	5700 4200 5800 4300
-Entry Wire Line
-	5700 4300 5800 4400
 $Comp
 L 1802ИР1 D60
@@
 Text HLabel 3700 9600 0    60   Input ~ 0
 XTAL
-Text Label 3400 9900 0    60   ~ 0
-MVI
 $Comp
 L CAP C4
@@
 Entry Wire Line
 	3300 9000 3400 9100
-Entry Wire Line
-	3300 9800 3400 9900
 $Comp
 L 556РТ4 D28
@@
 Entry Wire Line
 	10400 5800 10500 5900
-Entry Wire Line
-	10400 6100 10500 6200
 Wire Wire Line
 	4000 10800 3900 10800
@@
 	9400 5700 10400 5700
 Wire Wire Line
-	10200 6100 10400 6100
+	10200 6100 10250 6100
 Wire Wire Line
 	8500 5200 8800 5200
@@
 	5800 2500 6400 2500
 Wire Wire Line
-	6400 2600 5800 2600
-Wire Wire Line
 	5800 4300 6400 4300
-Wire Wire Line
-	6400 4400 5800 4400
 Wire Wire Line
 	6200 2800 6400 2800
@@
 Wire Wire Line
 	3700 9600 4000 9600
-Wire Wire Line
-	3400 9900 4000 9900
 Wire Wire Line
 	4000 9800 3900 9800
@@
 Wire Wire Line
 	3700 13200 4000 13200
+Text HLabel 10250 6100 2    60   Output ~ 0
+MVI
+Text HLabel 6200 2600 0    60   Input ~ 0
+MVI
+Wire Wire Line
+	6200 2600 6400 2600
+Text HLabel 6200 4400 0    60   Input ~ 0
+MVI
+Wire Wire Line
+	6200 4400 6400 4400
+Text HLabel 3700 9900 0    60   Input ~ 0
+MVI
+Wire Wire Line
+	3700 9900 4000 9900
 $EndSCHEMATC

Commit message: Cosmetic board fixes
Changed lines of the file:
@@
 	1    0    0    -1
 $EndComp
-Text Label 8200 5700 0    60   ~ 0
-HIGHT
 Text HLabel 8500 6200 0    60   Input ~ 0
 2M
@@
 $EndComp
 Entry Wire Line
-	8100 5600 8200 5700
-Entry Wire Line
 	10400 5700 10500 5800
 Entry Wire Line
@@
 Connection ~ 8700 5200
 Wire Wire Line
-	8200 5700 8800 5700
+	8500 5700 8800 5700
 Connection ~ 8600 5700
 Wire Wire Line
@@
 Wire Wire Line
 	3700 9900 4000 9900
+Text HLabel 8500 5700 0    60   Input ~ 0
+HIGHT
 $EndSCHEMATC
